Commit message: ik and obstacle

File: models/fr3_dual.urdf (robot description, URDF)
Before this commit: robot fr3, 45 links, 44 joints
Links:
- link base: geometry collision box size=0.6 1.4 0.05; visual box size=0.6 1.4 0.05
Joints:
- joint fr3_left_joint_base: origin xyz=0 0.405 1 rpy=0 0 0 -> xyz=0 0.405 0.05 rpy=0 0 0
- joint fr3_right_joint_base: origin xyz=0 -0.405 1 rpy=0 0 0 -> xyz=0 -0.405 0.05 rpy=0 0 0
